File: hardware/version001/fastLOGIC/fastLOGIC.kicad_pcb (KiCad board)
At the start: 2 copper layers, 60 x 92 mm, 82 parts, among them J1 AVR-ISP-6, J10 0-5V_ANALOG_IN_A, J11 PRES_SENS_BOTTOM, J12 PRES_SENS_TOP, J13 0-5V_ANALOG_IN_B, J14 RELAY_OUT_B, J15 RELAY_OUT_A, J3 DS18B20, J4 12-24V, J5 I2C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

Commit message: hardware minor mistake fixes
Parts:
- added R26: R4.7k, Resistor_SMD:R_0603_1608Metric, F.Cu at (45.0, 64.0)
- moved C15 3.83 mm to (40.8, 66.2), turned to 90 degrees
- moved C14 1.12 mm to (42.6, 64.8)
Connections:
- U5 pad 9: unconnected-(U5-~{RST}-Pad9) -> Net-(U5-~{RST})
Routing:
- net +12V: track 113.7 -> 127.2 mm
- net +5V: track 281.3 -> 290.6 mm
- net Net-(U5-~{RST}): track 0.00 -> 3.60 mm
- net GND: track 16.8 -> 19.8 mm, vias 226 -> 233
- net Net-(D5-A): track 14.2 -> 15.3 mm
- net Net-(J6-VBUS): track 18.8 -> 19.9 mm
Other:
- board text added: "by Jan Neumann 07.01.2024"
- board text removed: "by Jan Neumann 04.01.2024"
