File: hardware/version001/fastLOGIC/fastLOGIC.kicad_sch (KiCad schematic)
At the start: 82 parts, among them J1 AVR-ISP-6, J10 0-5V_ANALOG_IN_A, J11 PRES_SENS_BOTTOM, J12 PRES_SENS_TOP, J13 0-5V_ANALOG_IN_B, J14 RELAY_OUT_B, J15 RELAY_OUT_A, J3 DS18B20, J4 12-24V, J5 I2C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

Commit message: hardware minor mistake fixes
Parts:
- added R26: R4.7k, Resistor_SMD:R_0603_1608Metric, symbol Device:R
Connections:
- net +5V: now also R26.1
- net at U5.9 (~{RST}): now also R26.2
Changed lines of the file:
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@@
     (stroke (width 0) (type default))
   )
+  (wire (pts (xy 46.736 47.117) (xy 54.102 47.117))
+    (stroke (width 0) (type default))
+  )
   (wire (pts (xy 178.943 47.879) (xy 171.323 47.879))
     (stroke (width 0) (type default))
@@
     )
   )
+  (symbol (lib_id "power:+5V") (at 39.116 47.117 90) (unit 1)
+    (in_bom yes) (on_board yes) (dnp no)
+    (property "Reference" "#PWR016" (at 42.926 47.117 0)
+      (effects (font (size 1.27 1.27)) hide)
+    )
+    (property "Value" "+5V" (at 37.084 46.863 0)
+      (effects (font (size 1.27 1.27)) (justify left))
+    )
+    (property "Footprint" "" (at 39.116 47.117 0)
+      (effects (font (size 1.27 1.27)) hide)
+    )
+    (property "Datasheet" "" (at 39.116 47.117 0)
+      (effects (font (size 1.27 1.27)) hide)
+    )
+    (pin "1")
+    (instances
+      (project "fastLOGIC"
+        (path "/467e73ff-605e-4cd5-9b39-76afb3f5d14a"
+          (reference "#PWR016") (unit 1)
+        )
+      )
+    )
+  )
   (symbol (lib_id "power:GND") (at 209.804 261.747 180) (unit 1)
     (in_bom yes) (on_board yes) (dnp no)
@@
         )
       )
+    )
+  )
+  (symbol (lib_id "Device:R") (at 42.926 47.117 90) (unit 1)
+    (in_bom yes) (on_board yes) (dnp no) (fields_autoplaced)
+    (property "Reference" "R26" (at 42.926 42.418 90)
+      (effects (font (size 1.27 1.27)))
+    )
+    (property "Value" "R4.7k" (at 42.926 44.958 90)
+      (effects (font (size 1.27 1.27)))
+    )
+    (property "Footprint" "Resistor_SMD:R_0603_1608Metric" (at 42.926 48.895 90)
+      (effects (font (size 1.27 1.27)) hide)
+    )
+    (property "Datasheet" "~" (at 42.926 47.117 0)
+      (effects (font (size 1.27 1.27)) hide)
+    )
+    (property "LCSC" "C23162" (at 42.926 47.117 0)
+      (effects (font (size 1.27 1.27)) hide)
+    )
+    (pin "1")
+    (pin "2")
+    (instances
+      (project "fastLOGIC"
+        (path "/467e73ff-605e-4cd5-9b39-76afb3f5d14a"
+          (reference "R26") (unit 1)
+        )
+      )
